Commit message: feat(gimbal): wire dual-axis test setup for controller tuning

File: src/rm2_ecat/rm2_ecat_ros/urdf/test.urdf.xacro (robot description, xacro)
@@ -1,13 +1,23 @@
 <?xml version="1.0"?>
-<robot name="test_joint" xmlns:xacro="http://www.ros.org/wiki/xacro">
+<robot name="gimbal_test" xmlns:xacro="http://www.ros.org/wiki/xacro">
   <link name="base_link">
   </link>
-  <link name="test_link">
+  <link name="yaw_link">
   </link>
-  <joint name="test_joint" type="continuous">
+  <link name="pitch_link">
+  </link>
+  <joint name="yaw_motor" type="continuous">
     <parent link="base_link"/>
-    <child link="test_link"/>
+    <child link="yaw_link"/>
     <origin xyz="0 0 0.1" rpy="0 0 0"/>
     <axis xyz="0 0 1"/>
+    <limit lower="-1e10" upper="1e10" velocity="10.0" effort="5.0"/>
+    <dynamics damping="0.1" friction="0.01"/>
+  </joint>
+  <joint name="pitch_motor" type="continuous">
+    <parent link="yaw_link"/>
+    <child link="pitch_link"/>
+    <origin xyz="0 0 0.05" rpy="0 0 0"/>
+    <axis xyz="0 1 0"/>
     <limit lower="-1e10" upper="1e10" velocity="10.0" effort="5.0"/>
     <dynamics damping="0.1" friction="0.01"/>
@@ -17,5 +27,5 @@
       <plugin>rm2_ecat_ros/RmEcatHardwareInterface</plugin>
     </hardware>
-    <joint name="test_joint">
+    <joint name="yaw_motor">
       <command_interface name="effort"/>
       <state_interface name="position"/>
@@ -23,13 +33,31 @@
       <state_interface name="effort"/>
     </joint>
-    <transmission name="test_trans">
+    <joint name="pitch_motor">
+      <command_interface name="effort"/>
+      <state_interface name="position"/>
+      <state_interface name="velocity"/>
+      <state_interface name="effort"/>
+    </joint>
+    <transmission name="yaw_trans">
       <type>transmission_interface/SimpleTransmission</type>
       <plugin>transmission_interface/SimpleTransmission</plugin>
-      <joint name="test_joint" role="actuated">
+      <joint name="yaw_motor" role="actuated">
         <hardwareInterface>rm2_ecat_ros/RmEcatHardwareInterface</hardwareInterface>
         <mechanical_reduction>19.2032</mechanical_reduction>
         <offset>0.0</offset>
       </joint>
-      <actuator name="test_motor" role="actuated">
+      <actuator name="yaw_motor" role="actuated">
+        <mechanical_reduction>1</mechanical_reduction>
+      </actuator>
+    </transmission>
+    <transmission name="pitch_trans">
+      <type>transmission_interface/SimpleTransmission</type>
+      <plugin>transmission_interface/SimpleTransmission</plugin>
+      <joint name="pitch_motor" role="actuated">
+        <hardwareInterface>rm2_ecat_ros/RmEcatHardwareInterface</hardwareInterface>
+        <mechanical_reduction>19.2032</mechanical_reduction>
+        <offset>0.0</offset>
+      </joint>
+      <actuator name="pitch_motor" role="actuated">
         <mechanical_reduction>1</mechanical_reduction>
       </actuator>
